File: LED Controller/BC-250 LED Controller.kicad_sch (KiCad schematic)
At the start: 23 parts, among them J2000 BC-250 Micro Fit Connector, J3 BC-250 Power Btn Pins, J5 ATX Power Supply, SW1 Front_Panel_Power_Button (1 o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, SW2 Front_Panel_Power_Button (2 o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

Commit message: Fix LED Controller Schematic
I had the high and low power output LEDs/transistors labeled backwards on the schematic. Thanks to @elektricM for pointing this out!
Parts:
- renumbered Blue2_Control_Transitor to Blue1_Control_Transitor, Blue2_LED_High_Power to Blue1_LED_Low_Power, Blue1_Control_Transistor to Blue2_Control_Transistor, Blue1_LED_Low_Power to Blue2_LED_High_Power
Changed lines of the file:
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@@
 		(in_pos_files yes)
 		(dnp no)
-		(property "Reference" "Blue2_LED_High_Power"
+		(property "Reference" "Blue1_LED_Low_Power"
 			(at 133.096 79.756 0)
 			(show_name no)
@@
 			(project "BC-250 LED Controller"
 				(path "/020da3e5-9289-483e-acf0-9488f4973bf9"
-					(reference "Blue2_LED_High_Power")
+					(reference "Blue1_LED_Low_Power")
 					(unit 1)
 				)
@@
 		(in_pos_files yes)
 		(dnp no)
-		(property "Reference" "Blue2_Control_Transitor"
+		(property "Reference" "Blue1_Control_Transitor"
 			(at 133.35 58.4201 0)
 			(show_name no)
@@
 			(project "BC-250 LED Controller"
 				(path "/020da3e5-9289-483e-acf0-9488f4973bf9"
-					(reference "Blue2_Control_Transitor")
+					(reference "Blue1_Control_Transitor")
 					(unit 1)
 				)
@@
 		(in_pos_files yes)
 		(dnp no)
-		(property "Reference" "Blue1_Control_Transistor"
+		(property "Reference" "Blue2_Control_Transistor"
 			(at 49.53 58.4201 0)
 			(show_name no)
@@
 			(project "BC-250 LED Controller"
 				(path "/020da3e5-9289-483e-acf0-9488f4973bf9"
-					(reference "Blue1_Control_Transistor")
+					(reference "Blue2_Control_Transistor")
 					(unit 1)
 				)
@@
 		(in_pos_files yes)
 		(dnp no)
-		(property "Reference" "Blue1_LED_Low_Power"
+		(property "Reference" "Blue2_LED_High_Power"
 			(at 59.436 80.01 0)
 			(show_name no)
@@
 			(project "BC-250 LED Controller"
 				(path "/020da3e5-9289-483e-acf0-9488f4973bf9"
-					(reference "Blue1_LED_Low_Power")
+					(reference "Blue2_LED_High_Power")
 					(unit 1)
 				)
